Commit message: chore(Протестировал навигацию, лидар, одометрию, tf2)

File: src/autonomy_description/urdf/gazebo_plugins.xacro (robot description, xacro)
@@ -2,35 +2,43 @@
 <robot xmlns:xacro="http://www.ros.org/wiki/xacro">
     <xacro:macro name="gazebo_plugins">
-        <!-- ===================================================== -->
-        <!-- Gazebo visual properties                              -->
-        <!-- ===================================================== -->
+        <!-- ========================================================= -->
+        <!-- Materials / contact                                       -->
+        <!-- ========================================================= -->
         <gazebo reference="base_link">
             <material>Gazebo/Blue</material>
         </gazebo>
-        <gazebo reference="left_wheel_link">
-            <material>
-                Gazebo/Black
-            </material>
+        <!--
+            Four-wheel skid-steer.
+            Higher longitudinal friction and lower lateral friction
+            let the wheels roll normally while still allowing the robot
+            to skid sideways slightly during rotation.
+        -->
+        <gazebo reference="front_left_wheel_link">
+            <material>Gazebo/Black</material>
             <mu1>1.0</mu1>
-            <mu2>1.0</mu2>
+            <mu2>0.25</mu2>
             <kp>1000000.0</kp>
             <kd>100.0</kd>
         </gazebo>
-        <gazebo reference="right_wheel_link">
-            <material>
-                Gazebo/Black
-            </material>
+        <gazebo reference="front_right_wheel_link">
+            <material>Gazebo/Black</material>
             <mu1>1.0</mu1>
-            <mu2>1.0</mu2>
+            <mu2>0.25</mu2>
             <kp>1000000.0</kp>
             <kd>100.0</kd>
         </gazebo>
-        <!-- Caster should slide easily -->
-        <gazebo reference="caster_link">
-            <material>
-                Gazebo/Grey
-            </material>
-            <mu1>0.01</mu1>
-            <mu2>0.01</mu2>
+        <gazebo reference="rear_left_wheel_link">
+            <material>Gazebo/Black</material>
+            <mu1>1.0</mu1>
+            <mu2>0.25</mu2>
+            <kp>1000000.0</kp>
+            <kd>100.0</kd>
+        </gazebo>
+        <gazebo reference="rear_right_wheel_link">
+            <material>Gazebo/Black</material>
+            <mu1>1.0</mu1>
+            <mu2>0.25</mu2>
+            <kp>1000000.0</kp>
+            <kd>100.0</kd>
         </gazebo>
         <gazebo reference="lidar_link">
@@ -43,46 +51,92 @@
             <material>Gazebo/White</material>
         </gazebo>
-        <!-- ===================================================== -->
-        <!-- Differential drive                                    -->
-        <!-- ===================================================== -->
+        <!-- ========================================================= -->
+        <!-- Four wheel skid-steer drive                               -->
+        <!-- ========================================================= -->
         <gazebo>
             <plugin
-                name="diff_drive"
+                name="skid_steer_drive"
                 filename="libgazebo_ros_diff_drive.so">
+                <!-- ================================================= -->
+                <!-- ROS                                                -->
+                <!-- ================================================= -->
                 <ros>
                     <namespace>/</namespace>
+                    <!--
+                        ROS 2 gazebo_ros_diff_drive uses the standard
+                        cmd_vel and odom topics. Use remapping if custom
+                        names are required.
+                    -->
+                    <remapping>
+                        cmd_vel:=/cmd_vel
+                    </remapping>
+                    <remapping>
+                        odom:=/odom
+                    </remapping>
                 </ros>
-                <update_rate>
-                    50
-                </update_rate>
-                <!-- Wheels -->
+                <!-- ================================================= -->
+                <!-- Update rate                                       -->
+                <!-- ================================================= -->
+                <update_rate>50</update_rate>
+                <!-- ================================================= -->
+                <!-- Four wheels                                       -->
+                <!-- ================================================= -->
+                <num_wheel_pairs>2</num_wheel_pairs>
+                <!--
+                    Pair 1: front wheels
+                -->
                 <left_joint>
-                    left_wheel_joint
+                    front_left_wheel_joint
                 </left_joint>
                 <right_joint>
-                    right_wheel_joint
+                    front_right_wheel_joint
                 </right_joint>
-                <!-- Geometry -->
+                <!--
+                    Pair 2: rear wheels
+                -->
+                <left_joint>
+                    rear_left_wheel_joint
+                </left_joint>
+                <right_joint>
+                    rear_right_wheel_joint
+                </right_joint>
+                <!-- ================================================= -->
+                <!-- Geometry                                          -->
+                <!-- ================================================= -->
+                <!-- Front pair -->
                 <wheel_separation>
                     ${wheel_separation}
                 </wheel_separation>
+                <!-- Rear pair -->
+                <wheel_separation>
+                    ${wheel_separation}
+                </wheel_separation>
+                <!-- Front wheels -->
                 <wheel_diameter>
                     ${2.0 * wheel_radius}
                 </wheel_diameter>
-                <!-- Limits -->
+                <!-- Rear wheels -->
+                <wheel_diameter>
+                    ${2.0 * wheel_radius}
+                </wheel_diameter>
+                <!-- ================================================= -->
+                <!-- Motor limits                                      -->
+                <!-- ================================================= -->
                 <max_wheel_torque>
                     20.0
                 </max_wheel_torque>
                 <max_wheel_acceleration>
-                    2.0
+                    3.0
                 </max_wheel_acceleration>
-                <!-- ROS input -->
-                <command_topic>
-                    cmd_vel
-                </command_topic>
-                <!-- ROS odometry -->
-                <odometry_topic>
-                    odom
-                </odometry_topic>
+                <!-- ================================================= -->
+                <!-- Odometry                                          -->
+                <!-- ================================================= -->
+                <publish_odom>true</publish_odom>
+                <publish_odom_tf>true</publish_odom_tf>
+                <!--
+                    Wheel TF will be generated from /joint_states by
+                    robot_state_publisher instead.
+                -->
+                <publish_wheel_tf>false</publish_wheel_tf>
                 <odometry_frame>
                     odom
@@ -91,13 +145,29 @@
                     base_footprint
                 </robot_base_frame>
-                <publish_odom>
-                    true
-                </publish_odom>
-                <publish_odom_tf>
-                    true
-                </publish_odom_tf>
-                <publish_wheel_tf>
-                    true
-                </publish_wheel_tf>
+            </plugin>
+        </gazebo>
+        <!-- ========================================================= -->
+        <!-- Joint state publisher                                    -->
+        <!-- ========================================================= -->
+        <gazebo>
+            <plugin
+                name="joint_state_publisher"
+                filename="libgazebo_ros_joint_state_publisher.so">
+                <ros>
+                    <namespace>/</namespace>
+                </ros>
+                <update_rate>30</update_rate>
+                <joint_name>
+                    front_left_wheel_joint
+                </joint_name>
+                <joint_name>
+                    front_right_wheel_joint
+                </joint_name>
+                <joint_name>
+                    rear_left_wheel_joint
+                </joint_name>
+                <joint_name>
+                    rear_right_wheel_joint
+                </joint_name>
             </plugin>
         </gazebo>

File: src/autonomy_description/urdf/robot.urdf.xacro (robot description, xacro)
@@ -34,5 +34,5 @@
         name="wheel_mass"
         value="0.8"/>
-    <!-- Distance between left and right wheel centers -->
+    <!-- Left-right distance -->
     <xacro:property
         name="wheel_separation"
@@ -41,5 +41,5 @@
         name="wheel_y"
         value="${wheel_separation / 2.0}"/>
-    <!-- Distance between front and rear wheel centers -->
+    <!-- Front-rear distance -->
     <xacro:property
         name="wheel_base"
@@ -48,9 +48,5 @@
         name="wheel_x"
         value="${wheel_base / 2.0}"/>
-    <!-- Wheel center relative to base_link -->
-    <xacro:property
-        name="wheel_z"
-        value="${wheel_radius - base_center_z}"/>
-    <!-- wheel center relative to base_link -->
+    <!-- Relative to base_link -->
     <xacro:property
         name="wheel_z"
